File: Libre/Libre.kicad_sch (KiCad schematic)
At the start: 20 parts, among them J1 4.2inch E-Ink Display Module, J2 Micro_SD_Card, J3 Battery connector, SW1 UP, SW2 DOWN, SW3 PREVOUS, SW4 NEXT, SW5 HOME, SW6 SW_SPDT, U1 ESP32-S3-DEVKITC-1-N16R8, U2 MCP73831-2-OT, U3 AP2112K-3.3

Commit message: Day 2
Parts:
- C1, C2, C5: footprint (none) -> Capacitor_SMD:C_0603_1608Metric
- C3, C4: footprint (none) -> Capacitor_SMD:C_0805_2012Metric
- J1: footprint (none) -> Connector_PinHeader_2.54mm:PinHeader_1x08_P2.54mm_Vertical
- J2: footprint (none) -> Connector_Card:microSD_HC_Molex_104031-0811
- J3: footprint (none) -> Connector_JST:JST_PH_S2B-PH-K_1x02_P2.00mm_Horizontal
- R1, R2, R3: footprint (none) -> Resistor_SMD:R_0603_1608Metric
- SW1, SW2, SW3, SW4, SW5: footprint (none) -> Button_Switch_SMD:SW_SPST_TL3305A
- SW6: footprint (none) -> Button_Switch_SMD:SW_SPDT_CK_JS102011SAQN
- U1: footprint ESP32-S3-DEVKITC-1-N8R2:XCVR_ESP32-S3-DEVKITC-1-N8R2 -> Esp:XCVR_ESP32-S3-DEVKITC-1-N16R8V
Other:
- moved on the sheet: C1, C2, C3, C4, C5, J1, J2, J3, R1, R2, R3, SW1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

Commit message: CAD Change
Parts:
- added H1, H2, H3, H4: MountingHole, MountingHole:MountingHole_2.5mm, symbol Mechanical:MountingHole
